Commit message: Comparing velocity estimates derived from the 2 methods

File: rsc/A1/A1_modified_up_mod_sensored.urdf (robot description, URDF)
Before this commit: robot A1, 18 links, 17 joints
Links:
- removed link imu_link
- added link imu_parent
Joints:
- joint imu_joint: child imu_link -> imu_parent

Commit message: Full sim run 1

File: rsc/A1/A1_modified_up_mod_sensored.urdf (robot description, URDF)
Before this commit: robot A1, 18 links, 17 joints
Joints:
- joint FL_calf_joint: limit lower=-3.09653369433 upper=3.016297857297 effort=33.5 velocity=21 -> lower=-2.69653369433 upper=-0.916297857297 effort=33.5 velocity=21
- joint FL_hip_joint: limit lower=-3.102851455917 upper=3.102851455917 effort=33.5 velocity=21 -> lower=-0.802851455917 upper=0.802851455917 effort=33.5 velocity=21
- joint FL_thigh_joint: limit lower=-3.0471975512 upper=3.10879020479 effort=33.5 velocity=21 -> lower=-1.0471975512 upper=4.18879020479 effort=33.5 velocity=21
- joint FR_calf_joint: limit lower=-3.09653369433 upper=3.0916297857297 effort=33.5 velocity=21 -> lower=-2.69653369433 upper=-0.916297857297 effort=33.5 velocity=21
- joint FR_hip_joint: limit lower=-3.102851455917 upper=3.102851455917 effort=33.5 velocity=21 -> lower=-0.802851455917 upper=0.802851455917 effort=33.5 velocity=21
- joint FR_thigh_joint: limit lower=-3.1047197551 upper=3.10879020479 effort=33.5 velocity=21 -> lower=-1.0471975512 upper=4.18879020479 effort=33.5 velocity=21
- joint RL_calf_joint: limit lower=-3.09653369433 upper=3.0916297857297 effort=33.5 velocity=21 -> lower=-2.69653369433 upper=-0.916297857297 effort=33.5 velocity=21
- joint RL_hip_joint: axis 1 0 0 -> 0 0 1; limit lower=-3.02851455917 upper=3.022851455917 effort=33.5 velocity=21 -> lower=-0.802851455917 upper=0.802851455917 effort=33.5 velocity=21
- joint RL_thigh_joint: limit lower=-4.0471975512 upper=3.08879020479 effort=33.5 velocity=21 -> lower=-1.0471975512 upper=4.18879020479 effort=33.5 velocity=21
- joint RR_calf_joint: limit lower=-3.09653369433 upper=3.096297857297 effort=33.5 velocity=21 -> lower=-2.69653369433 upper=-0.916297857297 effort=33.5 velocity=21
- joint RR_hip_joint: axis 1 0 0 -> 0 0 1; limit lower=-3.102851455917 upper=3.102851455917 effort=33.5 velocity=21 -> lower=-0.802851455917 upper=0.802851455917 effort=33.5 velocity=21
- joint RR_thigh_joint: limit lower=-4.0471975512 upper=3.08879020479 effort=33.5 velocity=21 -> lower=-1.0471975512 upper=4.18879020479 effort=33.5 velocity=21

File: rsc/A1/A1_modified_up_mod_z.urdf (robot description, URDF)
Before this commit: robot A1, 18 links, 17 joints
Links:
- removed link imu_parent
Joints:
- removed joint imu_joint
- joint FL_hip_joint: axis 1 0 0 -> 0 0 1; origin xyz=0.1805 0.047 0 rpy=0 0 0 -> xyz=0 0.047 0.1805 rpy=0 0 0
- joint FL_thigh_joint: origin xyz=0 0.0838 0 rpy=0 0 0 -> xyz=0 0.0838 0 rpy=0 -1.57079632679 0
- joint FR_hip_joint: axis 1 0 0 -> 0 0 1; origin xyz=0.1805 -0.047 0 rpy=0 0 0 -> xyz=0 -0.047 0.1805 rpy=0 0 0
- joint FR_thigh_joint: origin xyz=0 -0.0838 0 rpy=0 0 0 -> xyz=0 -0.0838 0 rpy=0 -1.57079632679 0
- joint RL_hip_joint: axis 1 0 0 -> 0 0 1; limit lower=-0.1 upper=0.1 effort=33.5 velocity=21 -> lower=-0.802851455917 upper=0.802851455917 effort=33.5 velocity=21; origin xyz=-0.1805 0.047 0 rpy=0 0 0 -> xyz=0 0.047 -0.1805 rpy=0 0 0
- joint RL_thigh_joint: origin xyz=0 0.0838 0 rpy=0 0 0 -> xyz=0 0.0838 0 rpy=0 -1.57079632679 0
- joint RR_hip_joint: axis 1 0 0 -> 0 0 1; limit lower=-0.1 upper=0.1 effort=33.5 velocity=21 -> lower=-0.802851455917 upper=0.802851455917 effort=33.5 velocity=21; origin xyz=-0.1805 -0.047 0 rpy=0 0 0 -> xyz=0 -0.047 -0.1805 rpy=0 0 0
- joint RR_thigh_joint: origin xyz=0 -0.0838 0 rpy=0 0 0 -> xyz=0 -0.0838 0 rpy=0 -1.57079632679 0
