Commit message: Removing rear hip limits to revert to original URDF

File: rsc/A1/A1_modified_new.urdf (robot description, URDF)
Before this commit: robot A1, 18 links, 17 joints
Joints:
- joint RL_hip_joint: limit lower=-0.1 upper=0.1 effort=33.5 velocity=21 -> lower=-0.802851455917 upper=0.802851455917 effort=33.5 velocity=21
- joint RR_hip_joint: limit lower=-0.1 upper=0.1 effort=33.5 velocity=21 -> lower=-0.802851455917 upper=0.802851455917 effort=33.5 velocity=21

Commit message: Rearweight 4 does not give good default dynamics velocity tracking

File: rsc/A1/A1_modified_new.urdf (robot description, URDF)
Before this commit: robot A1, 18 links, 17 joints
Joints:
- joint RL_hip_joint: limit lower=-0.802851455917 upper=0.802851455917 effort=33.5 velocity=21 -> lower=-0.1 upper=0.1 effort=33.5 velocity=21
- joint RR_hip_joint: limit lower=-0.802851455917 upper=0.802851455917 effort=33.5 velocity=21 -> lower=-0.1 upper=0.1 effort=33.5 velocity=21
