Commit message: Jul24Sim1: First simulation with Go2 worked

File: rsc/A1/Go2_modified_1.urdf (robot description, URDF)
Before this commit: robot go2_description, 17 links, 16 joints
Links:
- added link imu_parent
- link trunk: geometry collision box size=0.3762 0.0935 0.114; visual mesh filename=dae/base.dae
Joints:
- added joint imu_joint: type fixed, parent trunk, child imu_parent, origin xyz=0 0 0.1 rpy=0 1.57079632679 0
